File: splitspace.kicad_pcb (KiCad board)
At the start: 2 copper layers, 159 parts, among them P1 USB_OTG, SW1 SW_RESET, SW10 SW_Z, SW11 SW_LSUP, SW12 SW_2, SW13 SW_W, SW14 SW_S, SW15 SW_X, SW16 SW_LALT, SW17 SW_F2, SW18 SW_3, SW19 SW_E, SW2 SW_ESC, SW20 SW_D, SW21 SW_C, SW22 SW_4, SW23 SW_R, SW24 SW_F, SW25 SW_V, SW26 SW_F4, SW27 SW_5, SW28 SW_T, SW29 SW_G, SW3 SW_TAB, SW30 SW_B, SW31 SW_SPACE, SW32 SW_6, SW33 SW_Y, SW34 SW_H, SW35 SW_N, SW36 SW_F3, SW37 SW_7, SW38 SW_U, SW39 SW_J, SW4 SW_CAPS, SW40 SW_M, SW41 SW_RALT, SW42 SW_8, SW43 SW_I, SW44 SW_K, SW45 SW_COMMA, SW46 SW_RSUP, SW47 SW_9, SW48 SW_O, SW49 SW_L, SW5 SW_LSHIFT, SW50 SW_FSTOP, SW51 SW_RCTRL, SW52 SW_0, SW53 SW_P, SW54 SW_COLON, SW55 SW_FSLASH, SW56 SW_MINUS, SW57 SW_BRKL, SW58 SW_QUOTE, SW59 SW_RSHIFT, SW6 SW_LCTRL, SW60 SW_PLUS, SW61 SW_BRKR, SW62 SW_ENTER, SW63 SW_F1, SW64 SW_BKSP1, SW65 SW_BKSP2, SW66 SW_BKSLASH, SW67 SW_LCTRL2, SW68 SW_LSUP2, SW69 SW_LALT2, SW7 SW_1, SW70 SW_SPACE2, SW71 SW_SPACE3, SW72 SW_F32, SW73 SW_RALT2, SW74 SW_RSUP2, SW75 SW_RCTRL2, SW76 SW_RSHIFT2, SW77 SW_BKSP22, SW8 SW_Q, SW9 SW_A, U1 ATmega32U4, U2 ISP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

Commit message: Finished?? No name on board
Parts:
- added G***: LOGO, newkeebs:logo, F.Cu at (126.5, 93.0)
- added G***: LOGO, newkeebs:logo, B.Cu at (320.0, 92.0)
- added HOLE: VAL**, hole:PKRHC, F.Cu at (105.2, 103.3)
- added HOLE: VAL**, hole:PKRHSL, F.Cu at (82.2, 131.9)
- added HOLE: VAL**, hole:PKRHSL, F.Cu at (363.0, 131.9)
- added HOLE: VAL**, hole:PKRH, F.Cu at (208.2, 122.4)
- added HOLE: VAL**, hole:PKRH, F.Cu at (340.1, 103.3)
- added HOLE: VAL**, hole:PKRH, F.Cu at (270.5, 160.6)
- added PB0 PF7: CONN_01X02, Pin_Headers:Pin_Header_Straight_1x02_Pitch2.54mm, B.Cu at (112.8, 94.2)
- C2, C4, C5, C6, C7, C8, D1, R1, R2, R3, R4, SW1: moved to B.Cu
- SW10, SW12, SW13, SW14, SW15, SW17, SW18, SW19, SW2, SW20, SW21, SW22, SW23, SW24, SW25, SW27, SW28, SW29, SW30, SW32, SW33, SW34, SW35, SW36, SW37, SW38, SW39, SW40, SW42, SW43, SW44, SW45, SW47, SW48, SW49, SW50, SW52, SW53, SW54, SW55, SW56, SW57, SW58, SW60, SW61, SW63, SW64, SW65, SW68, SW7, SW74, SW8, SW9: footprint Keyboard:CHERRY_PCB_100H -> newkeebs:CHERRY_PCB_100H_NOSS
- SW4: footprint Keyboard:CHERRY_PCB_175H -> newkeebs:CHERRY_PCB_175H_SIDE
- moved R4 327.1 mm to (83.8, 126.0)
- moved D1 321.4 mm to (84.2, 123.8), turned to 180 degrees
- moved C5 311.8 mm to (103.5, 131.8)
- moved C4 301.7 mm to (103.5, 130.2)
- moved C2 279.9 mm to (96.0, 91.8), turned to 90 degrees
- moved R1 277.5 mm to (138.5, 128.5), turned to 270 degrees
- moved C6 272.3 mm to (115.0, 113.8), turned to 180 degrees
- moved C8 260.5 mm to (107.0, 111.0), turned to 270 degrees
- moved C7 247.5 mm to (118.8, 122.5), turned to 90 degrees
- moved SW1 239.2 mm to (141.5, 132.2), turned to 90 degrees
- moved U2 183.8 mm to (120.5, 130.5), turned to 270 degrees
- moved U1 144.3 mm to (110.5, 122.7)
- moved C1 134.9 mm to (118.8, 144.2)
- moved Y1 134.5 mm to (122.5, 142.0), turned to 90 degrees
- moved C3 133.8 mm to (118.8, 136.8)
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Connections:
- C8 pad 1: Net-(C8-Pad1) -> Net-(C2-Pad2)
Routing:
- net /COL1: track 300.0 -> 96.0 mm, vias 2 -> 0
- net /COL14: track 107.0 -> 309.6 mm, vias 6 -> 2
- net /COL13: track 117.8 -> 312.5 mm
- net /COL11: track 66.9 -> 257.9 mm, vias 0 -> 2
- net /COL2: track 288.9 -> 112.3 mm
- net /COL12: track 126.5 -> 298.6 mm, vias 4 -> 2
- net Net-(C2-Pad2): track 0.00 -> 148.0 mm, vias 0 -> 8
- net /COL3: track 263.5 -> 135.3 mm, vias 4 -> 2
- net /COL8: track 169.3 -> 279.3 mm
- net GND: track 25.8 -> 122.4 mm, vias 2 -> 14
- net /COL4: track 247.8 -> 151.7 mm
- net /COL7: track 176.3 -> 262.9 mm
- net /COL9: track 208.3 -> 290.8 mm
- net /COL10: track 235.0 -> 312.1 mm
- net /ROW3: track 299.3 -> 361.8 mm, vias 2 -> 3
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- added copper zone on B.Cu, net GND
Other:
- board outline added: 285 x 97.6 mm
