File: splitspace.sch (KiCad schematic (older format))
At the start: 144 parts

Commit message: Last commit before moving everything, roll back to this if you need it
Parts:
- added D63, D66: D, Diodes_SMD:SOD-323, symbol D
- added SW63: SW_F1, Keyboard:CHERRY_PCB_100H, symbol SW_PUSH
- added SW66: SW_BKSLASH, Keyboard:CHERRY_PCB_100H, symbol SW_PUSH
- added SW67: SW_LCTRL2, Keyboard:CHERRY_PCB_150H, symbol SW_PUSH
- added SW68: SW_LSUP2, Keyboard:CHERRY_PCB_100H, symbol SW_PUSH
- added SW69: SW_LALT2, Keyboard:CHERRY_PCB_150H, symbol SW_PUSH
- added SW70: SW_SPACE2, Keyboard:CHERRY_PCB_625H, symbol SW_PUSH
- added SW71: SW_SPACE3, Keyboard:CHERRY_PCB_700H, symbol SW_PUSH
- added SW72: SW_F32, Keyboard:CHERRY_PCB_125H, symbol SW_PUSH
- added SW73: SW_RALT2, Keyboard:CHERRY_PCB_150H, symbol SW_PUSH
- added SW74: SW_RSUP2, Keyboard:CHERRY_PCB_100H, symbol SW_PUSH
- added SW75: SW_RCTRL2, Keyboard:CHERRY_PCB_150H, symbol SW_PUSH
- added SW76: SW_RSHIFT2, Keyboard:CHERRY_PCB_175H, symbol SW_PUSH
- added SW77: SW_BKSP22, Keyboard:CHERRY_PCB_200H, symbol SW_PUSH
- D1: renamed from D?; footprint LEDs:LED-3MM -> LEDs:LED_1206
- D10, D11, D12, D13, D14, D15, D16, D17, D18, D19, D2, D20, D21, D22, D23, D24, D25, D26, D27, D28, D29, D3, D30, D31, D32, D33, D34, D35, D36, D37, D38, D39, D4, D40, D41, D42, D43, D44, D45, D46, D47, D48, D49, D5, D50, D51, D52, D53, D54, D55, D56, D57, D58, D59, D6, D60, D61, D62, D64, D65, D7, D8, D9: renamed from D?; footprint (none) -> Diodes_SMD:SOD-323
- SW10: renamed from SW?; value SW_PUSH -> SW_Z; footprint (none) -> Keyboard:CHERRY_PCB_100H
- SW11: renamed from SW?; value SW_PUSH -> SW_LSUP; footprint (none) -> Keyboard:CHERRY_PCB_125H
- SW12: renamed from SW?; value SW_PUSH -> SW_2; footprint (none) -> Keyboard:CHERRY_PCB_100H
- SW13: renamed from SW?; value SW_PUSH -> SW_W; footprint (none) -> Keyboard:CHERRY_PCB_100H
- SW14: renamed from SW?; value SW_PUSH -> SW_S; footprint (none) -> Keyboard:CHERRY_PCB_100H
- SW15: renamed from SW?; value SW_PUSH -> SW_X; footprint (none) -> Keyboard:CHERRY_PCB_100H
- SW16: renamed from SW?; value SW_PUSH -> SW_LALT; footprint (none) -> Keyboard:CHERRY_PCB_125H
- SW17: renamed from SW?; value SW_PUSH -> SW_F2; footprint (none) -> Keyboard:CHERRY_PCB_100H
- SW18: renamed from SW?; value SW_PUSH -> SW_3; footprint (none) -> Keyboard:CHERRY_PCB_100H
- SW19: renamed from SW?; value SW_PUSH -> SW_E; footprint (none) -> Keyboard:CHERRY_PCB_100H
- SW2: renamed from SW?; value SW_PUSH -> SW_ESC; footprint (none) -> Keyboard:CHERRY_PCB_100H
- SW20: renamed from SW?; value SW_PUSH -> SW_D; footprint (none) -> Keyboard:CHERRY_PCB_100H
- SW21: renamed from SW?; value SW_PUSH -> SW_C; footprint (none) -> Keyboard:CHERRY_PCB_100H
- SW22: renamed from SW?; value SW_PUSH -> SW_4; footprint (none) -> Keyboard:CHERRY_PCB_100H
- SW23: renamed from SW?; value SW_PUSH -> SW_R; footprint (none) -> Keyboard:CHERRY_PCB_100H
- SW24: renamed from SW?; value SW_PUSH -> SW_F; footprint (none) -> Keyboard:CHERRY_PCB_100H
- SW25: renamed from SW?; value SW_PUSH -> SW_V; footprint (none) -> Keyboard:CHERRY_PCB_100H
- SW26: renamed from SW?; value SW_PUSH -> SW_F4; footprint (none) -> Keyboard:CHERRY_PCB_275H
- SW27: renamed from SW?; value SW_PUSH -> SW_5; footprint (none) -> Keyboard:CHERRY_PCB_100H
- SW28: renamed from SW?; value SW_PUSH -> SW_T; footprint (none) -> Keyboard:CHERRY_PCB_100H
- SW29: renamed from SW?; value SW_PUSH -> SW_G; footprint (none) -> Keyboard:CHERRY_PCB_100H
- SW3: renamed from SW?; value SW_PUSH -> SW_TAB; footprint (none) -> Keyboard:CHERRY_PCB_150H
- SW30: renamed from SW?; value SW_PUSH -> SW_B; footprint (none) -> Keyboard:CHERRY_PCB_100H
- SW31: renamed from SW?; value SW_PUSH -> SW_SPACE; footprint (none) -> Keyboard:CHERRY_PCB_275H
- SW32: renamed from SW?; value SW_PUSH -> SW_6; footprint (none) -> Keyboard:CHERRY_PCB_100H
- SW33: renamed from SW?; value SW_PUSH -> SW_Y; footprint (none) -> Keyboard:CHERRY_PCB_100H
- SW34: renamed from SW?; value SW_PUSH -> SW_H; footprint (none) -> Keyboard:CHERRY_PCB_100H
- SW35: renamed from SW?; value SW_PUSH -> SW_N; footprint (none) -> Keyboard:CHERRY_PCB_100H
- SW36: renamed from SW?; value SW_PUSH -> SW_F3; footprint (none) -> Keyboard:CHERRY_PCB_100H
- SW37: renamed from SW?; value SW_PUSH -> SW_7; footprint (none) -> Keyboard:CHERRY_PCB_100H
- SW38: renamed from SW?; value SW_PUSH -> SW_U; footprint (none) -> Keyboard:CHERRY_PCB_100H
- SW39: renamed from SW?; value SW_PUSH -> SW_J; footprint (none) -> Keyboard:CHERRY_PCB_100H
- SW4: renamed from SW?; value SW_PUSH -> SW_CAPS; footprint (none) -> Keyboard:CHERRY_PCB_175H
- SW40: renamed from SW?; value SW_PUSH -> SW_M; footprint (none) -> Keyboard:CHERRY_PCB_100H
- SW41: renamed from SW?; value SW_PUSH -> SW_RALT; footprint (none) -> Keyboard:CHERRY_PCB_125H
- SW42: renamed from SW?; value SW_PUSH -> SW_8; footprint (none) -> Keyboard:CHERRY_PCB_100H
- SW43: renamed from SW?; value SW_PUSH -> SW_I; footprint (none) -> Keyboard:CHERRY_PCB_100H
- SW44: renamed from SW?; value SW_PUSH -> SW_K; footprint (none) -> Keyboard:CHERRY_PCB_100H
- SW45: renamed from SW?; value SW_PUSH -> SW_COMMA; footprint (none) -> Keyboard:CHERRY_PCB_100H
- SW46: renamed from SW?; value SW_PUSH -> SW_RSUP; footprint (none) -> Keyboard:CHERRY_PCB_125H
- SW47: renamed from SW?; value SW_PUSH -> SW_9; footprint (none) -> Keyboard:CHERRY_PCB_100H
- SW48: renamed from SW?; value SW_PUSH -> SW_O; footprint (none) -> Keyboard:CHERRY_PCB_100H
- SW49: renamed from SW?; value SW_PUSH -> SW_L; footprint (none) -> Keyboard:CHERRY_PCB_100H
- SW5: renamed from SW?; value SW_PUSH -> SW_LSHIFT; footprint (none) -> Keyboard:CHERRY_PCB_225H
- SW50: renamed from SW?; value SW_PUSH -> SW_FSTOP; footprint (none) -> Keyboard:CHERRY_PCB_100H
- SW51: renamed from SW?; value SW_PUSH -> SW_RCTRL; footprint (none) -> Keyboard:CHERRY_PCB_125H
- SW52: renamed from SW?; value SW_PUSH -> SW_0; footprint (none) -> Keyboard:CHERRY_PCB_100H
- SW53: renamed from SW?; value SW_PUSH -> SW_P; footprint (none) -> Keyboard:CHERRY_PCB_100H
- SW54: renamed from SW?; value SW_PUSH -> SW_COLON; footprint (none) -> Keyboard:CHERRY_PCB_100H
- SW55: renamed from SW?; value SW_PUSH -> SW_FSLASH; footprint (none) -> Keyboard:CHERRY_PCB_100H
- SW56: renamed from SW?; value SW_PUSH -> SW_MINUS; footprint (none) -> Keyboard:CHERRY_PCB_100H
- SW57: renamed from SW?; value SW_PUSH -> SW_BRKL; footprint (none) -> Keyboard:CHERRY_PCB_100H
- SW58: renamed from SW?; value SW_PUSH -> SW_QUOTE; footprint (none) -> Keyboard:CHERRY_PCB_100H
- SW59: renamed from SW?; value SW_PUSH -> SW_RSHIFT; footprint (none) -> Keyboard:CHERRY_PCB_275H
- SW6: renamed from SW?; value SW_PUSH -> SW_LCTRL; footprint (none) -> Keyboard:CHERRY_PCB_125H
- SW60: renamed from SW?; value SW_PUSH -> SW_PLUS; footprint (none) -> Keyboard:CHERRY_PCB_100H
- SW61: renamed from SW?; value SW_PUSH -> SW_BRKR; footprint (none) -> Keyboard:CHERRY_PCB_100H
- SW62: renamed from SW?; value SW_PUSH -> SW_ENTER; footprint (none) -> Keyboard:CHERRY_PCB_225H
- SW64: renamed from SW?; value SW_PUSH -> SW_BKSP1; footprint (none) -> Keyboard:CHERRY_PCB_100H
- SW65: renamed from SW?; value SW_PUSH -> SW_BKSP2; footprint (none) -> Keyboard:CHERRY_PCB_100H
- SW7: renamed from SW?; value SW_PUSH -> SW_1; footprint (none) -> Keyboard:CHERRY_PCB_100H
- SW8: renamed from SW?; value SW_PUSH -> SW_Q; footprint (none) -> Keyboard:CHERRY_PCB_100H
- SW9: renamed from SW?; value SW_PUSH -> SW_A; footprint (none) -> Keyboard:CHERRY_PCB_100H
- U1: renamed from U?; footprint Housings_QFP:TQFP-44_10x10mm_Pitch0.8mm -> Keyboard:TQFP-44_10x10mm_Pitch0.8mm
- Y1: renamed from Y?; footprint Keyboards:HC49SM -> Keyboard:HC49SM
- gave numbers to parts that had none: 15
Connections:
- net COL13: now also D63.1 (K)
- net COL14: now also D66.1 (K)
- net ROW2: now also SW77.1
- net ROW3: now also SW66.1
- net ROW4: now also SW63.1, SW76.1
- net ROW5: now also SW67.1, SW68.1, SW69.1, SW70.1, SW71.1, SW72.1, SW73.1, SW74.1, SW75.1
- net at D6.2 (A), SW6.2: now also SW67.2
- net at D11.2 (A), SW11.2: now also SW68.2
- net at D16.2 (A), SW16.2: now also SW69.2
- net at D31.2 (A), SW31.2: now also SW70.2, SW71.2
- net at D36.2 (A), SW36.2: now also SW72.2
- net at D41.2 (A), SW41.2: now also SW73.2
- net at D46.2 (A), SW46.2: now also SW74.2
- net at D65.2 (A), SW65.2: now also SW77.2
- net at D59.2 (A), SW59.2: now also SW76.2
- net at D51.2 (A), SW51.2: now also SW75.2
- new net: D63.2 (A), SW63.2
- new net: D66.2 (A), SW66.2
- no-connect marks 1 -> 2

Commit message: Finished?? No name on board
Parts:
- added P2: CONN_01X02, Pin_Headers:Pin_Header_Straight_1x02_Pitch2.54mm, symbol CONN_01X02
- D1: symbol LED -> LED-RESCUE-splitspace
- P1: symbol USB_OTG -> USB_OTG-RESCUE-splitspace
- U1: symbol ATmega32U4 -> ATmega32U4-RESCUE-splitspace
Connections:
- wire segments 511 -> 512
Changed lines of the file:
@@
 EESchema Schematic File Version 2
+LIBS:splitspace-rescue
 LIBS:power
 LIBS:device
@@
 $EndDescr
 $Comp
-L USB_OTG P1
+L USB_OTG-RESCUE-splitspace P1
 U 1 1 576E0F9F
 P 1100 2050
@@
 $EndComp
 $Comp
-L LED D1
+L LED-RESCUE-splitspace D1
 U 1 1 576E0FB0
 P 5450 3550
@@
 $EndComp
 $Comp
-L ATmega32U4 U1
+L ATmega32U4-RESCUE-splitspace U1
 U 1 1 576E0F9E
 P 3750 3300
@@
 $EndComp
 NoConn ~ 4200 5000
+$Comp
+L CONN_01X02 P2
+U 1 1 5884B6BC
+P 6300 1900
+F 0 "P2" H 6300 2050 50  0000 C CNN
+F 1 "CONN_01X02" V 6400 1900 50  0000 C CNN
+F 2 "Pin_Headers:Pin_Header_Straight_1x02_Pitch2.54mm" H 6300 1900 50  0001 C CNN
+F 3 "" H 6300 1900 50  0000 C CNN
+	1    6300 1900
+	1    0    0    -1
+$EndComp
 Wire Wire Line
 	2100 1400 2100 2050
@@
 	1800 1400 1800 2250
 Connection ~ 2150 2050
-Connection ~ 2250 1950
 Connection ~ 2400 1850
 Wire Wire Line
@@
 	2450 4400 2150 4400
 Wire Wire Line
-	2250 4000 2550 4000
-Wire Wire Line
-	2250 2850 2250 4000
-Wire Wire Line
 	2200 1950 2500 1950
 Wire Wire Line
@@
 	5100 1950 5100 1050
 Wire Wire Line
-	4950 1950 5100 1950
-Wire Wire Line
 	3200 1050 3300 1050
 Wire Wire Line
@@
 	1950 3150 2500 3150
 Wire Wire Line
-	2250 1950 2250 2950
-Wire Wire Line
 	2200 2850 2500 2850
 Wire Wire Line
@@
 	2450 4500 2450 4550
 Wire Wire Line
-	2500 4350 2500 4300
-Wire Wire Line
-	2500 4300 2450 4300
-Wire Wire Line
 	2450 4400 2450 4450
 Wire Wire Line
-	2550 4250 2450 4250
-Wire Wire Line
-	2450 4250 2450 4300
-Wire Wire Line
-	2550 4000 2550 3950
-Wire Wire Line
 	2050 2900 2050 3150
 Wire Wire Line
@@
 	9700 2650 9700 2850
 Wire Wire Line
-	9850 3150 9600 3150
+	9600 3150 9850 3150
 Wire Wire Line
 	10300 3700 10350 3700
@@
 	9700 3500 9700 3700
 Wire Wire Line
-	9850 4000 9600 4000
+	9600 4000 9850 4000
 Wire Wire Line
 	10300 4550 10450 4550
@@
 	21400 2050 20950 2050
 Connection ~ 20950 2050
+Wire Wire Line
+	2550 4250 2550 4300
+Wire Wire Line
+	2550 4300 2450 4300
+Wire Wire Line
+	2450 4300 2450 4350
+Wire Wire Line
+	2550 3950 1900 3950
+Wire Wire Line
+	1900 3950 1900 1400
+Connection ~ 1900 1400
+Wire Wire Line
+	4950 1750 6100 1750
+Wire Wire Line
+	6100 1750 6100 1850
+Wire Wire Line
+	4950 1950 5100 1950
+Wire Wire Line
+	4950 4650 6100 4650
+Wire Wire Line
+	6100 4650 6100 1950
 $EndSCHEMATC
